Commit message: Adding launch file and rviz config file. Modifying the URDF

File: config/ura_config.urdf (robot description, URDF)
Before this commit: robot URA, 4 links, 3 joints
Links:
- removed link base
- added link base_link; visual cylinder length=0.03 radius=0.075
- added link base_plate; visual cylinder length=0.01 radius=0.075
- link tool: geometry visual box size=0.1 0.05 0.05
Joints:
- added joint top_rotation: type planar, parent bottom_arm, child top_arm, origin xyz=0.2 0 0 rpy=0 0 0, axis 1 0 0, limit lower=0 upper=1 effort=10 velocity=10
- joint base_rotation: child base -> base_plate; limit (none) -> lower=0 upper=1 effort=10 velocity=10; origin xyz=0 0 0 rpy=0 0 0 -> xyz=0 0 0.01 rpy=0 0 0; parent bottom_arm -> base_link
- joint bottom_rotation: limit (none) -> lower=0 upper=1 effort=10 velocity=10; origin xyz=0.06 0 0.045 rpy=0 0 0 -> xyz=0.16 0 0.045 rpy=0 0 0; parent top_arm -> base_plate
- joint tool_rotation: child top_arm -> tool; limit (none) -> lower=0 upper=1 effort=10 velocity=10; origin xyz=0.175 0 0 rpy=0 0 0 -> xyz=0.125 0 0 rpy=0 0 1.570796; parent tool -> top_arm

Commit message: Modifying URDF to get displacement with joint_state_publisher and adjust robot frame

File: config/ura_config.urdf (robot description, URDF)
Before this commit: robot URA, 5 links, 4 joints
Links:
- link base_link: geometry visual cylinder length=0.05 radius=0.075
Joints:
- joint base_rotation: limit lower=0 upper=1 effort=10 velocity=10 -> lower=-3.14 upper=3.14 effort=10 velocity=10; origin xyz=0 0 0.01 rpy=0 0 0 -> xyz=0 0 0.03 rpy=0 0 0; type planar -> revolute
- joint bottom_rotation: limit lower=0 upper=1 effort=10 velocity=10 -> lower=0 upper=-1.57 effort=10 velocity=10; origin xyz=0.16 0 0.045 rpy=0 0 0 -> xyz=0.03 0 0.045 rpy=0 0 0; type planar -> revolute
- joint tool_rotation: axis 0 0 1 -> 0 1 0; limit lower=0 upper=1 effort=10 velocity=10 -> lower=-3.14 upper=3.14 effort=10 velocity=10; type planar -> revolute
- joint top_rotation: axis 1 0 0 -> 0 1 0; limit lower=0 upper=1 effort=10 velocity=10 -> lower=-1.57 upper=1.57 effort=10 velocity=10; type planar -> revolute

Commit message: Adding launch file for Gazebo. Modifying URDF to fit Gazebo demand.

File: config/ura_config.urdf (robot description, URDF)
Before this commit: robot URA, 5 links, 4 joints
Links:
- link base_link: mass None -> 1; geometry collision cylinder length=0.05 radius=0.075; visual cylinder length=0.05 radius=0.075
- link base_plate: mass None -> 1; geometry collision cylinder length=0.01 radius=0.075; visual cylinder length=0.01 radius=0.075
- link bottom_arm: mass None -> 1; geometry collision box size=0.20 0.02 0.045; visual box size=0.20 0.02 0.045
- link tool: mass None -> 1; geometry collision box size=0.1 0.05 0.05; visual box size=0.1 0.05 0.05
- link top_arm: mass None -> 1; geometry collision box size=0.20 0.02 0.045; visual box size=0.20 0.02 0.045
Joints:
- joint bottom_rotation: limit lower=0 upper=-1.57 effort=10 velocity=10 -> lower=-1.57 upper=0.0 effort=10 velocity=10
