Commit message: Adding new URDF with realistic model

File: urdf/URA.urdf (robot description, URDF)
Before this commit: robot URA_1, 5 links, 4 joints
Links:
- removed link J1
- removed link J2
- removed link J3
- removed link J4
- removed link base
- added link J1_link, mass 0.736736484648281; collision mesh filename=package://proc_ura/meshes/J1.STL; visual mesh filename=package://proc_ura/meshes/J1.STL
- added link J2_link, mass 0.109734997075546; collision mesh filename=package://proc_ura/meshes/J2.STL; visual mesh filename=package://proc_ura/meshes/J2.STL
- added link J3_link, mass 0.530209842688532; collision mesh filename=package://proc_ura/meshes/J3.STL; visual mesh filename=package://proc_ura/meshes/J3.STL
- added link J4_link, mass 0.0825165692757006; collision mesh filename=package://proc_ura/meshes/J4.STL; visual mesh filename=package://proc_ura/meshes/J4.STL
- added link base_link, mass 0.0876288345931558; collision mesh filename=package://proc_ura/meshes/base.STL; visual mesh filename=package://proc_ura/meshes/base.STL
Joints:
- joint J1: axis 0 0 0 -> 0 1 0; child J1 -> J1_link; limit (none) -> lower=-3.14 upper=3.14 effort=10 velocity=10; parent base -> base_link; type fixed -> revolute
- joint J2: child J2 -> J2_link; limit (none) -> lower=-2.0 upper=2.0 effort=10 velocity=10; parent J1 -> J1_link; type continuous -> revolute
- joint J3: child J3 -> J3_link; limit (none) -> lower=-3.14 upper=1.5 effort=10 velocity=10; parent J2 -> J2_link; type continuous -> revolute
- joint J4: child J4 -> J4_link; limit (none) -> lower=-3.14 upper=3.14 effort=10 velocity=10; parent J3 -> J3_link; type continuous -> revolute

Commit message: Working simulation with URA real design

File: urdf/URA.urdf (robot description, URDF)
Before this commit: robot URA, 5 links, 4 joints
Links:
- removed link J1_link
- removed link J2_link
- removed link J3_link
- removed link J4_link
- added link bottom_link, mass 0.736736484648281; collision mesh filename=package://proc_ura/meshes/J1.STL; visual mesh filename=package://proc_ura/meshes/J1.STL
- added link mid_link, mass 0.109734997075546; collision mesh filename=package://proc_ura/meshes/J2.STL; visual mesh filename=package://proc_ura/meshes/J2.STL
- added link tool_link, mass 0.0825165692757006; collision mesh filename=package://proc_ura/meshes/J4.STL; visual mesh filename=package://proc_ura/meshes/J4.STL
- added link top_link, mass 0.530209842688532; collision mesh filename=package://proc_ura/meshes/J3.STL; visual mesh filename=package://proc_ura/meshes/J3.STL
- added link world_link; collision box size=0.2 0.13 0.05; visual box size=0.2 0.13 0.05
Joints:
- removed joint J1
- removed joint J2
- removed joint J3
- removed joint J4
- added joint base_joint: type fixed, parent world_link, child base_link, origin xyz=0 0 0 rpy=0 0 0, axis 0 0 1
- added joint base_rotation_joint: type revolute, parent base_link, child bottom_link, origin xyz=0 0 0.0235 rpy=1.5708 0 0, axis 0 1 0, limit lower=-3.14 upper=3.14 effort=10 velocity=10
- added joint bottom_joint: type revolute, parent bottom_link, child mid_link, origin xyz=0 0.058884 -0.060428 rpy=1.3239 0 0, axis 1 0 0, limit lower=-2.0 upper=2.0 effort=10 velocity=10
- added joint tool_joint: type revolute, parent top_link, child tool_link, origin xyz=0.01785 0 -0.17158 rpy=0.010467 1.5708 0, axis 1 0 0, limit lower=-3.14 upper=3.14 effort=10 velocity=10
- added joint top_joint: type revolute, parent mid_link, child top_link, origin xyz=0 0 -0.2032 rpy=1.2782 0 0, axis 1 0 0, limit lower=-3.14 upper=1.5 effort=10 velocity=10

Commit message: Dynamixel move but not as expected

File: urdf/URA.urdf (robot description, URDF)
Before this commit: robot URA, 6 links, 5 joints
Joints:
- joint base_rotation_joint: limit lower=-3.14 upper=3.14 effort=10 velocity=10 -> lower=0 upper=5.23 effort=10 velocity=10
- joint bottom_joint: limit lower=-2.0 upper=2.0 effort=10 velocity=10 -> lower=0 upper=5.23 effort=10 velocity=10
- joint tool_joint: limit lower=-3.14 upper=3.14 effort=10 velocity=10 -> lower=0 upper=5.23 effort=10 velocity=10
- joint top_joint: limit lower=-3.14 upper=1.5 effort=10 velocity=10 -> lower=0 upper=5.23 effort=10 velocity=10

Commit message: upgrade model

File: urdf/URA.urdf (robot description, URDF)
Before this commit: robot URA, 6 links, 5 joints
Joints:
- joint base_rotation_joint: origin xyz=0 0 0.0235 rpy=1.5708 0 0 -> xyz=0 0 0.0235 rpy=1.5708 0 0.5236
- joint bottom_joint: limit lower=0 upper=5.23 effort=10 velocity=10 -> lower=0 upper=4.0 effort=10 velocity=10; origin xyz=0 0.058884 -0.060428 rpy=1.3239 0 0 -> xyz=0 0.058884 -0.060428 rpy=5.54 0 0
- joint top_joint: limit lower=0 upper=5.23 effort=10 velocity=10 -> lower=0 upper=4.64 effort=10 velocity=10; origin xyz=0 0 -0.2032 rpy=1.2782 0 0 -> xyz=0 0 -0.2032 rpy=0 0 0

Commit message: Udgrade model

File: urdf/URA.urdf (robot description, URDF)
Before this commit: robot URA, 6 links, 5 joints
Joints:
- joint base_rotation_joint: origin xyz=0 0 0.0235 rpy=1.5708 0 0.5236 -> xyz=0 0 0.0235 rpy=1.5708 0 0.53
- joint bottom_joint: limit lower=0 upper=4.0 effort=10 velocity=10 -> lower=0 upper=5.23 effort=10 velocity=10; origin xyz=0 0.058884 -0.060428 rpy=5.54 0 0 -> xyz=0 0.058884 -0.060428 rpy=-1 0 0
- joint top_joint: limit lower=0 upper=4.64 effort=10 velocity=10 -> lower=0 upper=5.23 effort=10 velocity=10; origin xyz=0 0 -0.2032 rpy=0 0 0 -> xyz=0 0 -0.2032 rpy=-2.5 0 0

Commit message: safe

File: urdf/URA.urdf (robot description, URDF)
Before this commit: robot URA, 6 links, 5 joints
Links:
- removed link world_link
- added link clamp_link, mass 0.0884654244685185; collision mesh filename=package://proc_ura/meshes/clamp.STL; visual mesh filename=package://proc_ura/meshes/clamp.STL
- added link sub_link, mass 0.148202375101878; collision mesh filename=package://proc_ura/meshes/base.STL; visual mesh filename=package://proc_ura/meshes/base.STL
- link base_link: mass 0.0876288345931558 -> 0.0450140458134961; geometry collision mesh filename=package://proc_ura/meshes/Fix.STL; visual mesh filename=package://proc_ura/meshes/Fix.STL
- link bottom_link: mass 0.736736484648281 -> 0.207119682952531
- link mid_link: mass 0.109734997075546 -> 0.318160127525053
- link tool_link: mass 0.0825165692757006 -> 0.105976928601757
- link top_link: mass 0.530209842688532 -> 0.102709673564339
Joints:
- added joint clamp_joint: type revolute, parent tool_link, child clamp_link, origin xyz=0 0.064598 -0.022252 rpy=1.5708 8.3267E-16 -1.1082, axis 0 1 0, limit lower=0 upper=5.23 effort=10 velocity=10
- joint base_joint: axis 0 0 1 -> 0 0 0; origin xyz=0 0 0 rpy=0 0 0 -> xyz=0.015325 0 0.004025 rpy=1.5708 0 0; parent world_link -> sub_link
- joint base_rotation_joint: axis 0 1 0 -> 0 -1 0; origin xyz=0 0 0.0235 rpy=1.5708 0 0.53 -> xyz=0 0.02254 0 rpy=0 0 -3.1416
- joint bottom_joint: axis 1 0 0 -> 0 1 0; origin xyz=0 0.058884 -0.060428 rpy=-1 0 0 -> xyz=-0.042 -0.086849 0 rpy=1.5708 -5.093E-17 -0.49648
- joint tool_joint: axis 1 0 0 -> 0 1 0; origin xyz=0.01785 0 -0.17158 rpy=0.010467 1.5708 0 -> xyz=0.016924 0 -0.062 rpy=3.1416 -0.86421 1.5708
- joint top_joint: axis 1 0 0 -> 0 1 0; origin xyz=0 0 -0.2032 rpy=-2.5 0 0 -> xyz=0 0 0.1524 rpy=3.1416 -0.64087 -3.1416

Commit message: Final with 1 mbs. Need to change to 115200 for Jallaire Board

File: urdf/URA.urdf (robot description, URDF)
Before this commit: robot URA, 7 links, 6 joints
Joints:
- joint base_rotation_joint: origin xyz=0 0.02254 0 rpy=0 0 -3.1416 -> xyz=0 0.02254 0 rpy=0 2.625 -3.1416
- joint bottom_joint: axis 0 1 0 -> 0 -1 0; limit lower=0 upper=5.23 effort=10 velocity=10 -> lower=0.9 upper=4.39 effort=10 velocity=10; origin xyz=-0.042 -0.086849 0 rpy=1.5708 -5.093E-17 -0.49648 -> xyz=-0.042 -0.086849 0 rpy=1.5708 0 1.5708
- joint clamp_joint: limit lower=0 upper=5.23 effort=10 velocity=10 -> lower=0 upper=2.57 effort=10 velocity=10
- joint tool_joint: origin xyz=0.016924 0 -0.062 rpy=3.1416 -0.86421 1.5708 -> xyz=0.016924 0 -0.062 rpy=3.1416 2.615 1.5708
- joint top_joint: limit lower=0 upper=5.23 effort=10 velocity=10 -> lower=0.25 upper=4.5 effort=10 velocity=10; origin xyz=0 0 0.1524 rpy=3.1416 -0.64087 -3.1416 -> xyz=0 0 0.1524 rpy=3.1416 1.5708 -3.1416
